File: projects/PB-002 Covox Sound/kicad/Covox Sound.sch (KiCad schematic (older format))
At the start: 43 parts, among them J1 Port A, J2 TRS_3.5mm, J3 Port B, J4 Signals, Q1 2N3904, SW1 SW_Push, SW2 SW_Push, SW3 SW_Push, SW4 SW_Push, SW5 SW_Push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

Commit message: Make a tone
Other:
- note removed: "A 4x4 LED Cube with integrated template, created for slotting on top of the RC-ONE\nProject Board. As a cube it's rather small, but given that it already contains 64 individual\nLEDs I believe it's a manageable yet fun project.\n\nEach layer is constructed separately on the reverse side with 0.5mm diameter metal bars\nfor the anodes. Layers are then moved to the front and stacked."
Changed lines of the file:
@@
 LIBS:contrib
 LIBS:valves
+LIBS:trs_3.5mm
+LIBS:rc1_backplane
 LIBS:mounting
-LIBS:trs_3.5mm
 LIBS:Covox Sound-cache
 EELAYER 25 0
@@
 	1    0    0    -1
 $EndComp
-Text Notes 11825 10550 0    60   ~ 0
-A 4x4 LED Cube with integrated template, created for slotting on top of the RC-ONE\nProject Board. As a cube it's rather small, but given that it already contains 64 individual\nLEDs I believe it's a manageable yet fun project.\n\nEach layer is constructed separately on the reverse side with 0.5mm diameter metal bars\nfor the anodes. Layers are then moved to the front and stacked.
 $Comp
 L Conn_01x10 J1
