File: platforms/PP 6502 Game Board/PP 6502 Game Board.sch (KiCad schematic (older format))
At the start: 33 parts, among them J1 BASE, J2 BTM, J3 TOP, J4 SBC, J5 TRS_3.5mm, M1 Mounting, M2 Mounting, M3 Mounting, M4 Mounting, Q1 2N2222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

Commit message: Gerber export
Other:
- note added: "Rodney Zaks wrote a whole book of games for the SYM-1 and I wanted to build it for\nuse with my computers as well. so this board takes care of the logic needed for a\n6502 or 6800 based computer. Also requires the game board project fitted on top as\nit contains all of the interactive parts needed."
Changed lines of the file:
@@
 encoding utf-8
 Sheet 1 1
-Title "ACIA"
+Title "6502 Game Board (PP)"
 Date ""
 Rev "A"
@@
 	-1   0    0    -1
 $EndComp
+Text Notes 11850 10375 0    60   ~ 0
+Rodney Zaks wrote a whole book of games for the SYM-1 and I wanted to build it for\nuse with my computers as well. so this board takes care of the logic needed for a\n6502 or 6800 based computer. Also requires the game board project fitted on top as\nit contains all of the interactive parts needed.
 $EndSCHEMATC
