File: projects/GB-001 Game Board/kicad/Game Board.sch (KiCad schematic (older format))
At the start: 48 parts, among them J1 TOP, J2 BTM, SW1 0, SW10 9, SW11 A, SW12 B, SW13 C, SW14 D, SW15 E, SW16 F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

Commit message: Gerber export
Other:
- note added: "6502 Game Board only slots into 6502 Game Board (PP). Somewhat limiting and not\nexactly what this repository was for, but Rodney Zaks wrote a whole book of games\nfor the SYM-1 and I wanted to build it for the RC-ONE instead. The logic is placed\nbelow on the Project Platform board (PP)."
Changed lines of the file:
@@
 LIBS:sw_keyboard
 LIBS:Game Board-cache
-LIBS:PP 6502 Game Board-cache
 EELAYER 25 0
 EELAYER END
@@
 encoding utf-8
 Sheet 1 1
-Title "ACIA"
+Title "6502 Game Board"
 Date ""
 Rev "A"
@@
 	1    0    0    -1
 $EndComp
+Text Notes 11875 10375 0    60   ~ 0
+6502 Game Board only slots into 6502 Game Board (PP). Somewhat limiting and not\nexactly what this repository was for, but Rodney Zaks wrote a whole book of games\nfor the SYM-1 and I wanted to build it for the RC-ONE instead. The logic is placed\nbelow on the Project Platform board (PP).
 $EndSCHEMATC
